File: kicad_diagram/kicad_diagram/kicad_diagram.kicad_sch (KiCad schematic)
At the start: 19 parts, among them U1 ESP32-CAM, U2 ESP32-CAM Programmer

Commit message: Tactics
Connections:
- net +5V: now also SERVO-MOTOR.2 (+); no longer SERVO-MOTOR.1 (PWM)
- net SERVO_PIN: now also SERVO-MOTOR.1 (PWM); no longer SERVO-MOTOR.2 (+)
- net +9V renamed +7.2V
Changed lines of the file:
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@@
 	(wire
 		(pts
-			(xy 215.9 24.13) (xy 215.9 41.91)
+			(xy 39.37 52.07) (xy 39.37 53.34)
 		)
 		(stroke
@@
 	(wire
 		(pts
-			(xy 35.56 48.26) (xy 35.56 53.34)
+			(xy 215.9 24.13) (xy 215.9 41.91)
 		)
 		(stroke
@@
 	(wire
 		(pts
-			(xy 40.64 54.61) (xy 40.64 52.07)
+			(xy 91.44 143.51) (xy 93.98 143.51)
 		)
 		(stroke
@@
 	(wire
 		(pts
-			(xy 91.44 143.51) (xy 93.98 143.51)
+			(xy 53.34 151.13) (xy 59.69 151.13)
 		)
 		(stroke
@@
 	(wire
 		(pts
-			(xy 53.34 151.13) (xy 59.69 151.13)
+			(xy 46.99 48.26) (xy 46.99 50.8)
 		)
 		(stroke
@@
 	(wire
 		(pts
-			(xy 46.99 48.26) (xy 46.99 50.8)
+			(xy 58.42 125.73) (xy 58.42 120.65)
 		)
 		(stroke
@@
 	(wire
 		(pts
-			(xy 58.42 125.73) (xy 58.42 120.65)
+			(xy 40.64 168.91) (xy 39.37 168.91)
 		)
 		(stroke
@@
 	(wire
 		(pts
-			(xy 40.64 168.91) (xy 39.37 168.91)
+			(xy 39.37 52.07) (xy 38.1 52.07)
 		)
 		(stroke
@@
 	(wire
 		(pts
-			(xy 109.22 80.01) (xy 111.76 80.01)
-		)
-		(stroke
-			(width 0)
-			(type default)
-		)
-	)
-	(wire
-		(pts
-			(xy 67.31 132.08) (xy 76.2 132.08)
+			(xy 38.1 52.07) (xy 38.1 48.26)
 		)
 		(stroke
@@
 	(wire
 		(pts
-			(xy 261.62 132.08) (xy 265.43 132.08)
+			(xy 109.22 80.01) (xy 111.76 80.01)
 		)
 		(stroke
@@
 	(wire
 		(pts
-			(xy 215.9 52.07) (xy 215.9 63.5)
+			(xy 67.31 132.08) (xy 76.2 132.08)
 		)
 		(stroke
@@
 	(wire
 		(pts
-			(xy 40.64 52.07) (xy 38.1 52.07)
+			(xy 261.62 132.08) (xy 265.43 132.08)
 		)
 		(stroke
@@
 	(wire
 		(pts
-			(xy 38.1 52.07) (xy 38.1 48.26)
+			(xy 215.9 52.07) (xy 215.9 63.5)
 		)
 		(stroke
@@
 	(wire
 		(pts
+			(xy 35.56 52.07) (xy 35.56 48.26)
+		)
+		(stroke
+			(width 0)
+			(type default)
+		)
+	)
+	(wire
+		(pts
 			(xy 234.95 132.08) (xy 240.03 132.08)
 		)
@@
 	(global_label "SERVO_PIN"
 		(shape input)
-		(at 40.64 54.61 270)
+		(at 35.56 52.07 270)
 		(fields_autoplaced yes)
 		(effects
@@
 		)
 		(property "Intersheetrefs" "${INTERSHEET_REFS}"
-			(at 40.64 67.8157 90)
+			(at 35.56 65.2757 90)
 			(effects
 				(font
@@
 	(symbol
 		(lib_id "power:+5V")
-		(at 35.56 53.34 180)
+		(at 39.37 53.34 180)
 		(unit 1)
 		(exclude_from_sim no)
@@
 		(fields_autoplaced yes)
 		(property "Reference" "#PWR08"
-			(at 35.56 49.53 0)
+			(at 39.37 49.53 0)
 			(effects
 				(font
@@
 		)
 		(property "Value" "+5V"
-			(at 35.56 58.42 0)
+			(at 39.37 58.42 0)
 			(effects
 				(font
@@
 		)
 		(property "Footprint" ""
-			(at 35.56 53.34 0)
+			(at 39.37 53.34 0)
 			(effects
 				(font
@@
 		)
 		(property "Datasheet" ""
-			(at 35.56 53.34 0)
+			(at 39.37 53.34 0)
 			(effects
 				(font
@@
 		)
 		(property "Description" "Power symbol creates a global label with name \"+5V\""
-			(at 35.56 53.34 0)
+			(at 39.37 53.34 0)
 			(effects
 				(font
@@
 			)
 		)
-		(property "Value" "+9V"
-			(at 240.03 143.51 0)
+		(property "Value" "+7.2V"
+			(at 242.57 139.6999 0)
 			(effects
 				(font
 					(size 1.27 1.27)
 				)
+				(justify right)
 			)
 		)
@@
 			)
 		)
-		(property "Value" "+9V"
+		(property "Value" "+7.2V"
 			(at 184.15 24.13 90)
 			(effects
